Commit message: fix urdf handler

File: urdf/SO_5DOF_ARM100_05d.SLDASM/urdf/SO_5DOF_ARM100_05d.SLDASM_fixed.urdf (robot description, URDF)
Before this commit: robot SO_5DOF_ARM100_05d.SLDASM, 7 links, 6 joints
Links:
- link Base: geometry collision mesh filename=../meshes/Base.STL; visual mesh filename=../meshes/Base.STL
- link Fixed_Gripper: geometry collision mesh filename=../meshes/Fixed_Gripper.STL; visual mesh filename=../meshes/Fixed_Gripper.STL
- link Lower_Arm: geometry collision mesh filename=../meshes/Lower_Arm.STL; visual mesh filename=../meshes/Lower_Arm.STL
- link Moving_Jaw: geometry collision mesh filename=../meshes/Moving_Jaw.STL; visual mesh filename=../meshes/Moving_Jaw.STL
- link Shoulder_Rotation_Pitch: geometry collision mesh filename=../meshes/Shoulder_Rotation_Pitch.STL; visual mesh filename=../meshes/Shoulder_Rotation_Pitch.STL
- link Upper_Arm: geometry collision mesh filename=../meshes/Upper_Arm.STL; visual mesh filename=../meshes/Upper_Arm.STL
- link Wrist_Pitch_Roll: geometry collision mesh filename=../meshes/Wrist_Pitch_Roll.STL; visual mesh filename=../meshes/Wrist_Pitch_Roll.STL
